File: design/eagle/fri3d_badge_2016.sch (EAGLE design)
At the start: 40 parts, among them K1 65100516121, Q1 MOSFET-NCHANNEL2N7002PW, U1 MCP73831

Commit message: added header for Analog pins A0-5
Parts:
- added U$2: HEADER-06X1-MALE, GeekAmmo:HEADER-06X1-MALE
Connections:
- new net A0: U$1.PF7(ADC7), U$2.6
- new net A1: U$1.PF6(ADC6), U$2.5
- new net A2: U$1.PF5(ADC5), U$2.4
- new net A3: U$1.PF4(ADC4), U$2.3
- new net A4: U$1.PF1(ADC1), U$2.2
- new net A5: U$1.PF0(ADC0), U$2.1
Other:
- moved on the sheet: ICSP, J3
Changed lines of the file:
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@@
 <part name="J3" library="SparkFun-Connectors" deviceset="M02" device="JST-PTH-VERT"/>
 <part name="K1" library="Input-Output_Connectors_rev15d" deviceset="65100516121" device=""/>
+<part name="U$2" library="GeekAmmo" deviceset="HEADER-06X1?" device="-MALE"/>
 </parts>
 <sheets>
@@
 <instance part="R3" gate="G$1" x="17.78" y="91.44" rot="R270"/>
 <instance part="C1" gate="G$1" x="25.4" y="91.44"/>
-<instance part="GND3" gate="1" x="5.08" y="58.42"/>
+<instance part="GND3" gate="1" x="-15.24" y="58.42"/>
 <instance part="GND4" gate="1" x="-33.02" y="86.36"/>
 <instance part="C2" gate="G$1" x="-33.02" y="91.44"/>
@@
 <instance part="S1" gate="G$1" x="185.42" y="149.86"/>
 <instance part="D2" gate="G$1" x="198.12" y="116.84" rot="R270"/>
-<instance part="ICSP" gate="A" x="-2.54" y="30.48"/>
+<instance part="ICSP" gate="A" x="-17.78" y="35.56"/>
 <instance part="GND9" gate="1" x="152.4" y="60.96"/>
 <instance part="SUPPLY4" gate="G$1" x="213.36" y="73.66"/>
@@
 <instance part="U$3" gate="G$1" x="71.12" y="27.94"/>
 <instance part="SUPPLY7" gate="G$1" x="104.14" y="33.02"/>
-<instance part="SUPPLY8" gate="G$1" x="12.7" y="35.56"/>
-<instance part="GND18" gate="1" x="12.7" y="22.86"/>
+<instance part="SUPPLY8" gate="G$1" x="-2.54" y="40.64"/>
+<instance part="GND18" gate="1" x="-2.54" y="27.94"/>
 <instance part="LED5" gate="G$1" x="-22.86" y="96.52"/>
 <instance part="R10" gate="G$1" x="-15.24" y="88.9"/>
@@
 <instance part="LED4" gate="G$1" x="205.74" y="25.4" rot="R270"/>
 <instance part="Q2" gate="G$1" x="63.5" y="96.52" rot="R90"/>
-<instance part="J3" gate="G$1" x="-10.16" y="63.5"/>
+<instance part="J3" gate="G$1" x="-30.48" y="63.5"/>
 <instance part="K1" gate="G$1" x="-22.86" y="134.62" rot="R180"/>
+<instance part="U$2" gate="G$1" x="20.32" y="35.56"/>
 </instances>
 <busses>
@@
 <segment>
 <pinref part="GND3" gate="1" pin="GND"/>
-<wire x1="5.08" y1="63.5" x2="5.08" y2="60.96" width="0.1524" layer="91"/>
+<wire x1="-15.24" y1="63.5" x2="-15.24" y2="60.96" width="0.1524" layer="91"/>
 <pinref part="J3" gate="G$1" pin="1"/>
-<wire x1="5.08" y1="63.5" x2="-2.54" y2="63.5" width="0.1524" layer="91"/>
+<wire x1="-15.24" y1="63.5" x2="-22.86" y2="63.5" width="0.1524" layer="91"/>
 </segment>
 <segment>
@@
 </segment>
 <segment>
-<wire x1="12.7" y1="27.94" x2="12.7" y2="25.4" width="0.1524" layer="91"/>
+<wire x1="-2.54" y1="33.02" x2="-2.54" y2="30.48" width="0.1524" layer="91"/>
 <pinref part="GND18" gate="1" pin="GND"/>
 <pinref part="ICSP" gate="A" pin="6"/>
-<wire x1="2.54" y1="27.94" x2="12.7" y2="27.94" width="0.1524" layer="91"/>
+<wire x1="-12.7" y1="33.02" x2="-2.54" y2="33.02" width="0.1524" layer="91"/>
 </segment>
 <segment>
@@
 </segment>
 <segment>
-<label x="0" y="66.04" size="1.778" layer="95"/>
+<label x="-20.32" y="66.04" size="1.778" layer="95"/>
 <pinref part="J3" gate="G$1" pin="2"/>
-<wire x1="5.08" y1="66.04" x2="-2.54" y2="66.04" width="0.1524" layer="91"/>
+<wire x1="-15.24" y1="66.04" x2="-22.86" y2="66.04" width="0.1524" layer="91"/>
 </segment>
 <segment>
@@
 <segment>
 <pinref part="ICSP" gate="A" pin="2"/>
-<wire x1="2.54" y1="33.02" x2="12.7" y2="33.02" width="0.1524" layer="91"/>
-<wire x1="12.7" y1="33.02" x2="12.7" y2="35.56" width="0.1524" layer="91"/>
+<wire x1="-12.7" y1="38.1" x2="-2.54" y2="38.1" width="0.1524" layer="91"/>
+<wire x1="-2.54" y1="38.1" x2="-2.54" y2="40.64" width="0.1524" layer="91"/>
 <pinref part="SUPPLY8" gate="G$1" pin="VCC"/>
 </segment>
@@
 <segment>
 <pinref part="ICSP" gate="A" pin="4"/>
-<wire x1="2.54" y1="30.48" x2="17.78" y2="30.48" width="0.1524" layer="91"/>
-<label x="12.7" y="30.48" size="1.778" layer="95"/>
+<wire x1="-12.7" y1="35.56" x2="2.54" y2="35.56" width="0.1524" layer="91"/>
+<label x="-2.54" y="35.56" size="1.778" layer="95"/>
 </segment>
 <segment>
@@
 <segment>
 <pinref part="ICSP" gate="A" pin="5"/>
-<wire x1="-5.08" y1="27.94" x2="-20.32" y2="27.94" width="0.1524" layer="91"/>
-<label x="-20.32" y="27.94" size="1.778" layer="95"/>
+<wire x1="-20.32" y1="33.02" x2="-35.56" y2="33.02" width="0.1524" layer="91"/>
+<label x="-35.56" y="33.02" size="1.778" layer="95"/>
 </segment>
 <segment>
@@
 <segment>
 <pinref part="ICSP" gate="A" pin="3"/>
-<wire x1="-5.08" y1="30.48" x2="-20.32" y2="30.48" width="0.1524" layer="91"/>
-<label x="-20.32" y="30.48" size="1.778" layer="95"/>
+<wire x1="-20.32" y1="35.56" x2="-35.56" y2="35.56" width="0.1524" layer="91"/>
+<label x="-35.56" y="35.56" size="1.778" layer="95"/>
 </segment>
 <segment>
@@
 <segment>
 <pinref part="ICSP" gate="A" pin="1"/>
-<wire x1="-5.08" y1="33.02" x2="-20.32" y2="33.02" width="0.1524" layer="91"/>
-<label x="-20.32" y="33.02" size="1.778" layer="95"/>
+<wire x1="-20.32" y1="38.1" x2="-35.56" y2="38.1" width="0.1524" layer="91"/>
+<label x="-35.56" y="38.1" size="1.778" layer="95"/>
 </segment>
 <segment>
@@
 </segment>
 </net>
+<net name="A0" class="0">
+<segment>
+<pinref part="U$1" gate="G$1" pin="PF7(ADC7)"/>
+<wire x1="106.68" y1="144.78" x2="142.24" y2="144.78" width="0.1524" layer="91"/>
+<label x="139.7" y="144.78" size="1.778" layer="95"/>
+</segment>
+<segment>
+<pinref part="U$2" gate="G$1" pin="6"/>
+<wire x1="25.4" y1="40.64" x2="35.56" y2="40.64" width="0.1524" layer="91"/>
+<label x="33.02" y="40.64" size="1.778" layer="95"/>
+</segment>
+</net>
+<net name="A1" class="0">
+<segment>
+<pinref part="U$1" gate="G$1" pin="PF6(ADC6)"/>
+<wire x1="106.68" y1="142.24" x2="142.24" y2="142.24" width="0.1524" layer="91"/>
+<label x="139.7" y="142.24" size="1.778" layer="95"/>
+</segment>
+<segment>
+<pinref part="U$2" gate="G$1" pin="5"/>
+<wire x1="25.4" y1="38.1" x2="35.56" y2="38.1" width="0.1524" layer="91"/>
+<label x="33.02" y="38.1" size="1.778" layer="95"/>
+</segment>
+</net>
+<net name="A2" class="0">
+<segment>
+<pinref part="U$1" gate="G$1" pin="PF5(ADC5)"/>
+<wire x1="106.68" y1="139.7" x2="142.24" y2="139.7" width="0.1524" layer="91"/>
+<label x="139.7" y="139.7" size="1.778" layer="95"/>
+</segment>
+<segment>
+<pinref part="U$2" gate="G$1" pin="4"/>
+<wire x1="25.4" y1="35.56" x2="35.56" y2="35.56" width="0.1524" layer="91"/>
+<label x="33.02" y="35.56" size="1.778" layer="95"/>
+</segment>
+</net>
+<net name="A3" class="0">
+<segment>
+<pinref part="U$1" gate="G$1" pin="PF4(ADC4)"/>
+<wire x1="106.68" y1="137.16" x2="142.24" y2="137.16" width="0.1524" layer="91"/>
+<label x="139.7" y="137.16" size="1.778" layer="95"/>
+</segment>
+<segment>
+<pinref part="U$2" gate="G$1" pin="3"/>
+<wire x1="25.4" y1="33.02" x2="35.56" y2="33.02" width="0.1524" layer="91"/>
+<label x="33.02" y="33.02" size="1.778" layer="95"/>
+</segment>
+</net>
+<net name="A4" class="0">
+<segment>
+<pinref part="U$1" gate="G$1" pin="PF1(ADC1)"/>
+<wire x1="106.68" y1="134.62" x2="142.24" y2="134.62" width="0.1524" layer="91"/>
+<label x="139.7" y="134.62" size="1.778" layer="95"/>
+</segment>
+<segment>
+<pinref part="U$2" gate="G$1" pin="2"/>
+<wire x1="25.4" y1="30.48" x2="35.56" y2="30.48" width="0.1524" layer="91"/>
+<label x="33.02" y="30.48" size="1.778" layer="95"/>
+</segment>
+</net>
+<net name="A5" class="0">
+<segment>
+<pinref part="U$1" gate="G$1" pin="PF0(ADC0)"/>
+<wire x1="106.68" y1="132.08" x2="142.24" y2="132.08" width="0.1524" layer="91"/>
+<label x="139.7" y="132.08" size="1.778" layer="95"/>
+</segment>
+<segment>
+<pinref part="U$2" gate="G$1" pin="1"/>
+<wire x1="25.4" y1="27.94" x2="35.56" y2="27.94" width="0.1524" layer="91"/>
+<label x="33.02" y="27.94" size="1.778" layer="95"/>
+</segment>
+</net>

Commit message: fixed IR receiver and button Arduino pins
Parts:
- added R18: 10K, SparkFun-Passives:RESISTOR0805-RES
Connections:
- net BUTTON: now also R18.1, S1.2, U$1.PD2(RX); no longer S1.1, U$1.PD6(ADC9)
- net GND: now also R18.2
- net IR_RX: now also U$1.PD3(TX); no longer U$1.PD5
- net N$3: now also S1.1; no longer S1.2
Other:
- moved on the sheet: C8, S1
Changed lines of the file:
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@@
 <part name="K1" library="Input-Output_Connectors_rev15d" deviceset="65100516121" device=""/>
 <part name="U$2" library="GeekAmmo" deviceset="HEADER-06X1?" device="-MALE"/>
+<part name="R18" library="SparkFun-Passives" deviceset="RESISTOR" device="0805-RES" value="10K"/>
+<part name="GND10" library="SparkFun-Aesthetics" deviceset="GND" device=""/>
 </parts>
 <sheets>
@@
 <instance part="C6" gate="G$1" x="55.88" y="93.98" rot="R90"/>
 <instance part="GND8" gate="1" x="45.72" y="96.52" rot="R270"/>
-<instance part="S1" gate="G$1" x="185.42" y="149.86"/>
+<instance part="S1" gate="G$1" x="185.42" y="160.02" rot="R180"/>
 <instance part="D2" gate="G$1" x="198.12" y="116.84" rot="R270"/>
 <instance part="ICSP" gate="A" x="-17.78" y="35.56"/>
@@
 <instance part="R10" gate="G$1" x="-15.24" y="88.9"/>
 <instance part="C7" gate="G$1" x="99.06" y="25.4"/>
-<instance part="C8" gate="G$1" x="185.42" y="157.48" rot="R90"/>
+<instance part="C8" gate="G$1" x="186.436" y="149.86" rot="R90"/>
 <instance part="R12" gate="G$1" x="193.04" y="71.12"/>
 <instance part="R13" gate="G$1" x="193.04" y="55.88"/>
@@
 <instance part="K1" gate="G$1" x="-22.86" y="134.62" rot="R180"/>
 <instance part="U$2" gate="G$1" x="20.32" y="35.56"/>
+<instance part="R18" gate="G$1" x="167.64" y="147.32" rot="R270"/>
+<instance part="GND10" gate="1" x="167.64" y="139.7"/>
 </instances>
 <busses>
@@
 <junction x="-15.24" y="147.32"/>
 </segment>
+<segment>
+<pinref part="GND10" gate="1" pin="GND"/>
+<pinref part="R18" gate="G$1" pin="2"/>
+</segment>
 </net>
 <net name="D+" class="0">
@@
 <pinref part="U$1" gate="G$1" pin="PD0(SCL)"/>
 <wire x1="106.68" y1="114.3" x2="142.24" y2="114.3" width="0.1524" layer="91"/>
-<label x="137.16" y="114.3" size="1.778" layer="95"/>
+<label x="134.62" y="114.3" size="1.778" layer="95"/>
 </segment>
 </net>
 <net name="BUTTON" class="0">
 <segment>
-<pinref part="S1" gate="G$1" pin="1"/>
-<wire x1="180.34" y1="149.86" x2="175.26" y2="149.86" width="0.1524" layer="91"/>
 <wire x1="175.26" y1="149.86" x2="175.26" y2="154.94" width="0.1524" layer="91"/>
-<label x="160.02" y="154.94" size="1.778" layer="95"/>
+<label x="149.86" y="154.94" size="1.778" layer="95"/>
+<wire x1="175.26" y1="154.94" x2="167.64" y2="154.94" width="0.1524" layer="91"/>
+<wire x1="167.64" y1="154.94" x2="149.86" y2="154.94" width="0.1524" layer="91"/>
+<junction x="175.26" y="154.94"/>
+<pinref part="R18" gate="G$1" pin="1"/>
+<wire x1="167.64" y1="152.4" x2="167.64" y2="154.94" width="0.1524" layer="91"/>
+<junction x="167.64" y="154.94"/>
 <pinref part="C8" gate="G$1" pin="1"/>
-<wire x1="175.26" y1="154.94" x2="160.02" y2="154.94" width="0.1524" layer="91"/>
-<wire x1="180.34" y1="157.48" x2="175.26" y2="157.48" width="0.1524" layer="91"/>
-<wire x1="175.26" y1="157.48" x2="175.26" y2="154.94" width="0.1524" layer="91"/>
-<junction x="175.26" y="154.94"/>
-</segment>
-<segment>
-<pinref part="U$1" gate="G$1" pin="PD6(ADC9)"/>
-<wire x1="106.68" y1="91.44" x2="142.24" y2="91.44" width="0.1524" layer="91"/>
-<label x="132.08" y="91.44" size="1.778" layer="95"/>
+<wire x1="175.26" y1="149.86" x2="181.356" y2="149.86" width="0.1524" layer="91"/>
+<pinref part="S1" gate="G$1" pin="2"/>
+<wire x1="175.26" y1="154.94" x2="175.26" y2="160.02" width="0.1524" layer="91"/>
+<wire x1="175.26" y1="160.02" x2="180.34" y2="160.02" width="0.1524" layer="91"/>
+</segment>
+<segment>
+<pinref part="U$1" gate="G$1" pin="PD2(RX)"/>
+<wire x1="106.68" y1="121.92" x2="142.24" y2="121.92" width="0.1524" layer="91"/>
+<label x="132.08" y="121.92" size="1.778" layer="95"/>
 </segment>
 </net>
@@
 </segment>
 <segment>
-<pinref part="U$1" gate="G$1" pin="PD5"/>
-<wire x1="106.68" y1="73.66" x2="142.24" y2="73.66" width="0.1524" layer="91"/>
-<label x="137.16" y="73.66" size="1.778" layer="95"/>
+<pinref part="U$1" gate="G$1" pin="PD3(TX)"/>
+<wire x1="106.68" y1="119.38" x2="142.24" y2="119.38" width="0.1524" layer="91"/>
+<label x="134.62" y="119.38" size="1.778" layer="95"/>
 </segment>
 </net>
@@
 <net name="N$3" class="0">
 <segment>
-<pinref part="S1" gate="G$1" pin="2"/>
-<wire x1="190.5" y1="149.86" x2="195.58" y2="149.86" width="0.1524" layer="91"/>
 <wire x1="195.58" y1="149.86" x2="195.58" y2="154.94" width="0.1524" layer="91"/>
-<pinref part="C8" gate="G$1" pin="2"/>
-<wire x1="187.96" y1="157.48" x2="195.58" y2="157.48" width="0.1524" layer="91"/>
-<wire x1="195.58" y1="157.48" x2="195.58" y2="154.94" width="0.1524" layer="91"/>
 <pinref part="R5" gate="G$1" pin="1"/>
 <wire x1="195.58" y1="154.94" x2="200.66" y2="154.94" width="0.1524" layer="91"/>
 <junction x="195.58" y="154.94"/>
-</segment>
-</net>
+<pinref part="C8" gate="G$1" pin="2"/>
+<wire x1="188.976" y1="149.86" x2="195.58" y2="149.86" width="0.1524" layer="91"/>
+<pinref part="S1" gate="G$1" pin="1"/>
+<wire x1="190.5" y1="160.02" x2="195.58" y2="160.02" width="0.1524" layer="91"/>
+<wire x1="195.58" y1="160.02" x2="195.58" y2="154.94" width="0.1524" layer="91"/>
+</segment>
+</net>

Commit message: added switch and draft silkscreen
Parts:
- added S2: (no value), SparkFun-Electromechanical:SWITCH-SPDT-SMD-A
Connections:
- new net N$17: J3.2, S2.P
- net VCC: now also S2.S; no longer J3.2
Changed lines of the file:
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@@
 <part name="R18" library="SparkFun-Passives" deviceset="RESISTOR" device="0805-RES" value="10K"/>
 <part name="GND10" library="SparkFun-Aesthetics" deviceset="GND" device=""/>
+<part name="S2" library="SparkFun-Electromechanical" deviceset="SWITCH-SPDT" device="-SMD-A"/>
 </parts>
 <sheets>
@@
 <instance part="R18" gate="G$1" x="167.64" y="147.32" rot="R270"/>
 <instance part="GND10" gate="1" x="167.64" y="139.7"/>
+<instance part="S2" gate="1" x="-7.62" y="66.04"/>
 </instances>
 <busses>
@@
 </segment>
 <segment>
-<label x="-20.32" y="66.04" size="1.778" layer="95"/>
-<pinref part="J3" gate="G$1" pin="2"/>
-<wire x1="-15.24" y1="66.04" x2="-22.86" y2="66.04" width="0.1524" layer="91"/>
-</segment>
-<segment>
 <pinref part="SUPPLY2" gate="G$1" pin="VCC"/>
 <pinref part="R4" gate="G$1" pin="1"/>
@@
 <wire x1="215.9" y1="154.94" x2="215.9" y2="160.02" width="0.1524" layer="91"/>
 </segment>
+<segment>
+<pinref part="S2" gate="1" pin="S"/>
+<wire x1="-2.54" y1="63.5" x2="7.62" y2="63.5" width="0.1524" layer="91"/>
+</segment>
 </net>
 <net name="N$5" class="0">
@@
 </segment>
 </net>
+<net name="N$17" class="0">
+<segment>
+<pinref part="J3" gate="G$1" pin="2"/>
+<pinref part="S2" gate="1" pin="P"/>
+<wire x1="-22.86" y1="66.04" x2="-12.7" y2="66.04" width="0.1524" layer="91"/>
+<wire x1="-12.7" y1="66.04" x2="-10.16" y2="66.04" width="0.1524" layer="91"/>
+</segment>
+</net>

Commit message: changed resistors on RGB LED to 220 (to test)
Parts:
- R16, R17, R7, R8, R9: value 22 -> 220
Changed lines of the file:
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@@
 <part name="SUPPLY4" library="SparkFun-Aesthetics" deviceset="VCC" device=""/>
 <part name="SUPPLY5" library="SparkFun-Aesthetics" deviceset="VCC" device=""/>
-<part name="R7" library="SparkFun-Passives" deviceset="RESISTOR" device="0805-RES" value="22"/>
-<part name="R8" library="SparkFun-Passives" deviceset="RESISTOR" device="0805-RES" value="22"/>
+<part name="R7" library="SparkFun-Passives" deviceset="RESISTOR" device="0805-RES" value="220"/>
+<part name="R8" library="SparkFun-Passives" deviceset="RESISTOR" device="0805-RES" value="220"/>
 <part name="SUPPLY6" library="SparkFun-Aesthetics" deviceset="VCC" device=""/>
 <part name="GND17" library="SparkFun-Aesthetics" deviceset="GND" device=""/>
@@
 <part name="R6" library="SparkFun-Passives" deviceset="RESISTOR" device="0805-RES" value="220"/>
 <part name="R11" library="SparkFun-Passives" deviceset="RESISTOR" device="0805-RES" value="220"/>
-<part name="R9" library="SparkFun-Passives" deviceset="RESISTOR" device="0805-RES" value="22"/>
-<part name="R16" library="SparkFun-Passives" deviceset="RESISTOR" device="0805-RES" value="22"/>
-<part name="R17" library="SparkFun-Passives" deviceset="RESISTOR" device="0805-RES" value="22"/>
+<part name="R9" library="SparkFun-Passives" deviceset="RESISTOR" device="0805-RES" value="220"/>
+<part name="R16" library="SparkFun-Passives" deviceset="RESISTOR" device="0805-RES" value="220"/>
+<part name="R17" library="SparkFun-Passives" deviceset="RESISTOR" device="0805-RES" value="220"/>
 <part name="LED1" library="led" deviceset="LED" device="CHIPLED_0805"/>
 <part name="LED2" library="led" deviceset="LED" device="CHIPLED_0805"/>
